File: yoradio-2/yoradio-2.kicad_pcb (KiCad board)
At the start: 2 copper layers, 160 x 55 mm, 50 parts, among them J1 Conn_01x04, J2 Conn_01x04, J3 AudioJack2_Dual_Ground_Switch, J4 Conn_01x02, J5 Conn_01x03, J6 Conn_01x04, J7 Conn_01x01, M3 TPS63020, Q1 IRF7404, Q2 BC858R

Commit message: Add files via upload
Parts:
- added C16: 10n, Capacitor_SMD:C_1206_3216Metric_Pad1.33x1.80mm_HandSolder, B.Cu at (226.2, 96.2)
- added Q3: IRF7404, Package_SO:SOIC-8_3.9x4.9mm_P1.27mm, B.Cu at (220.1, 97.5)
- added R8: 47k, Resistor_SMD:R_1206_3216Metric, B.Cu at (227.6, 99.8)
- added R9: 220, Resistor_SMD:R_1206_3216Metric, B.Cu at (208.3, 100.2)
- C1: value 0.1u -> 1u
- moved R5 2.03 mm to (212.4, 95.5), turned to 180 degrees
Connections:
- M4 pad 6: /BAT_OUT+ -> Net-(J4-Pin_2)
Routing:
- net Net-(J4-Pin_2): track 6.29 -> 29.2 mm
- net Net-(Q3-G): track 0.00 -> 21.1 mm, vias 0 -> 2
- net +USB_C: track 36.9 -> 39.4 mm
- net /BAT_OUT+: track 63.3 -> 61.2 mm
- net GND: vias 8 -> 9
