File: yoradio-2/yoradio-2.kicad_sch (KiCad schematic)
At the start: 51 parts, among them J1 Conn_01x04, J2 Conn_01x04, J3 AudioJack2_Dual_Ground_Switch, J4 Conn_01x02, J5 Conn_01x03, J6 Conn_01x04, J7 Conn_01x01, M3 TPS63020, Q1 IRF7404, Q2 BC858R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

Commit message: Add files via upload
Parts:
- added C16: 10n, Capacitor_SMD:C_1206_3216Metric_Pad1.33x1.80mm_HandSolder, symbol Device:C_Small
- added Q3: IRF7404, Package_SO:SOIC-8_3.9x4.9mm_P1.27mm, symbol Transistor_FET:IRF7404
- added R8: 47k, Resistor_SMD:R_1206_3216Metric, symbol Device:R_Small
- added R9: 220, Resistor_SMD:R_1206_3216Metric, symbol Device:R_Small
- C1: value 0.1u -> 1u
Connections:
- net +USB_C: now also R9.2
- net BAT_OUT+: now also C16.2, Q3.1 (S), Q3.2 (S), Q3.3 (S); no longer M4.6 (___OUT+)
- net GND: now also R8.1
- net at J4.2 (Pin_2), M4.5 (___BATTERY+), M6.1 (+BATT): now also M4.6 (___OUT+), Q3.5 (D), Q3.6 (D), Q3.7 (D), Q3.8 (D)
- new net: C16.1, Q3.4 (G), R8.2, R9.1
Other:
- moved on the sheet: C10, C13, C15, C5, C6, C7, C8, C9, M3
