File: JFET-amp-gramofon/JFET-amp-gramofon.kicad_pcb (KiCad board)
At the start: 2 copper layers, 52 x 40 mm, 32 parts, among them J2 DIN-5, J3 Conn_01x02, J4 Conn_01x01_Pin, J5 Conn_01x01_Pin, J6 Conn_01x03, Q1 BF245A, Q2 BF245A, U2 LM78L12_TO92

Commit message: Add files via upload
Parts:
- removed REF** (x2): MountingHole_2mm, MountingHole:MountingHole_2mm
- added C5: 470n, Capacitor_SMD:C_0805_2012Metric, B.Cu at (108.3, 95.3)
- added C6: 470n, Capacitor_SMD:C_0805_2012Metric, B.Cu at (108.2, 90.8)
- J2: moved to B.Cu
- R1, R2: value 2M2 -> 1M
- R10, R9: value 22k -> 91k
- R11, R12: value 22k -> 10k
- U2: value LM78L12_TO92 -> LM78L09_TO92
- moved R2 1.65 mm to (105.5, 85.4)
- moved Q1 0.84 mm to (112.0, 96.1)
- moved R1 0.41 mm to (104.4, 100.5)
- moved Q2 0.23 mm to (112.5, 89.9)
- turned J2 to -90 degrees
Connections:
- net +12V renamed +9V
- J2 pad 1: Net-(J2-Pad1) -> unconnected-(J2-Pad1)
- J2 pad 2: Net-(J2-Pad2) -> unconnected-(J2-Pad2)
- J2 pad 4: unconnected-(J2-Pad4) -> Net-(J2-Pad4)
- J2 pad 5: unconnected-(J2-Pad5) -> Net-(J2-Pad5)
- Q1 pad 1: Net-(J6-Pin_1) -> Net-(Q1-G)
- Q2 pad 1: Net-(J6-Pin_3) -> Net-(Q2-G)
- R1 pad 1: Net-(J6-Pin_1) -> Net-(Q1-G)
- R10 pad 2: Net-(J2-Pad2) -> Net-(J2-Pad4)
- R11 pad 1: Net-(J2-Pad1) -> Net-(J2-Pad5)
- R12 pad 2: Net-(J2-Pad2) -> Net-(J2-Pad4)
- R2 pad 1: Net-(J6-Pin_3) -> Net-(Q2-G)
- R9 pad 2: Net-(J2-Pad1) -> Net-(J2-Pad5)
Routing:
- net Net-(J2-Pad4): track 0.00 -> 17.5 mm, vias 0 -> 1
- net Net-(J2-Pad2): track 17.5 -> 0.00 mm, vias 1 -> 0
- net Net-(J6-Pin_1): track 18.5 -> 4.63 mm
- net Net-(J2-Pad5): track 0.00 -> 13.0 mm, vias 0 -> 1
- net Net-(J2-Pad1): track 13.0 -> 0.00 mm, vias 1 -> 0
- net Net-(Q1-G): track 0.00 -> 9.52 mm
- net Net-(Q2-G): track 0.00 -> 9.46 mm
- net Net-(J6-Pin_3): track 13.0 -> 4.89 mm
- net Net-(Q1-D): track 13.6 -> 7.77 mm
- net Net-(Q1-S): track 12.4 -> 13.7 mm
