File: JFET-amp-gramofon/JFET-amp-gramofon.kicad_sch (KiCad schematic)
At the start: 30 parts, among them J2 DIN-5, J3 Conn_01x02, J4 Conn_01x01_Pin, J5 Conn_01x01_Pin, J6 Conn_01x03, Q1 BF245A, Q2 BF245A, U2 LM78L12_TO92

Commit message: Add files via upload
Parts:
- added C5, C6: 470n, Capacitor_SMD:C_0805_2012Metric, symbol Device:C_Small
- R1, R2: value 2M2 -> 1M
- R10, R9: value 22k -> 91k
- R11, R12: value 22k -> 10k
- U2: value LM78L12_TO92 -> LM78L09_TO92
Connections:
- net at Q1.1 (G), R1.1: now also C5.2; no longer J6.1 (Pin_1)
- net at R10.2, R12.2: now also J2.4; no longer J2.2
- net at R11.1, R9.2: now also J2.5; no longer J2.1
- net at Q2.1 (G), R2.1: now also C6.2; no longer J6.3 (Pin_3)
- net +12V renamed +9V
- new net: C5.1, J6.1 (Pin_1)
- new net: C6.1, J6.3 (Pin_3)
Other:
- moved on the sheet: J4, R1, R2, R3, R4, R5, RV2
